File: Kicad_Oscillator_Drone.sch (KiCad schematic (older format))
At the start: 57 parts, among them J1 Power Out, J10 AudioJack, J11 AudioJack, J12 AudioJack, J14 AudioJack, J15 AudioJack, J17 AudioJack, J2 Power Out, J3 Jack-DC, J6 AudioJack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

Commit message: Vactrol and pwr fix
Power fix and alteration
Remove LFO1 AM
Add Vactrol to OSC1
Net names
Parts:
- added D?: OSC1CV, LED_THT:LED_D3.0mm, symbol Device:LED
- added J?: OSC1CV, Connector_Audio:AudioJack3StereoNarrow-PJ-321, symbol Connector:AudioJack3_Ground
- added R?: OSC1CV, OptoDevice:R_LDR_10x8.5mm_P7.6mm_Vertical, symbol Sensor_Optical:LDR03
- added R?: 1k2, Resistor_SMD:R_0805_2012Metric_Pad1.15x1.40mm_HandSolder, symbol Device:R
- C1: footprint Capacitor_THT:CP_Radial_D7.5mm_P2.50mm -> Capacitor_THT:CP_Radial_D6.3mm_P2.50mm
- J3: footprint Connector_BarrelJack:BarrelJack_CUI_PJ-102AH_Horizontal -> Connector_BarrelJack:BarrelJack_CUI_PJ-063AH_Horizontal
- RV1: Position (none) -> LFO1
- RV3: Pos (none) -> LFO1
Connections:
- net labels added: DC-in, OSC1-CV
- wire segments 151 -> 159
Changed lines of the file:
@@
 	9525 1875 9525 1775
 Wire Wire Line
-	9525 1775 8950 1775
+	9525 1775 9300 1775
 Connection ~ 8950 1775
 Wire Wire Line
@@
 L power:+10V #PWR0103
 U 1 1 5C12E6A4
-P 1500 1000
-F 0 "#PWR0103" H 1500 850 50  0001 C CNN
-F 1 "+10V" H 1515 1173 50  0000 C CNN
-F 2 "" H 1500 1000 50  0001 C CNN
-F 3 "" H 1500 1000 50  0001 C CNN
-	1    1500 1000
+P 2075 1050
+F 0 "#PWR0103" H 2075 900 50  0001 C CNN
+F 1 "+10V" H 2090 1223 50  0000 C CNN
+F 2 "" H 2075 1050 50  0001 C CNN
+F 3 "" H 2075 1050 50  0001 C CNN
+	1    2075 1050
 	1    0    0    -1
 $EndComp
@@
 F 0 "C1" H 1618 1321 50  0000 L CNN
 F 1 "100u" H 1618 1230 50  0000 L CNN
-F 2 "Capacitor_THT:CP_Radial_D7.5mm_P2.50mm" H 1538 1125 50  0001 C CNN
+F 2 "Capacitor_THT:CP_Radial_D6.3mm_P2.50mm" H 1538 1125 50  0001 C CNN
 F 3 "~" H 1500 1275 50  0001 C CNN
 	1    1500 1275
@@
 Wire Notes Line
 	550  2000 550  600
-Wire Wire Line
-	1500 1000 1500 1050
 $Comp
 L Connector:Jack-DC J3
@@
 F 0 "J3" H 905 1600 50  0000 C CNN
 F 1 "Jack-DC" H 905 1509 50  0000 C CNN
-F 2 "Connector_BarrelJack:BarrelJack_CUI_PJ-102AH_Horizontal" H 900 1235 50  0001 C CNN
+F 2 "Connector_BarrelJack:BarrelJack_CUI_PJ-063AH_Horizontal" H 900 1235 50  0001 C CNN
 F 3 "~" H 900 1235 50  0001 C CNN
 	1    850  1275
@@
 L power:PWR_FLAG #FLG0101
 U 1 1 5C1318B3
-P 1150 1050
-F 0 "#FLG0101" H 1150 1125 50  0001 C CNN
-F 1 "PWR_FLAG" H 1150 1224 50  0000 C CNN
-F 2 "" H 1150 1050 50  0001 C CNN
-F 3 "~" H 1150 1050 50  0001 C CNN
-	1    1150 1050
-	1    0    0    -1
-$EndComp
-Connection ~ 1150 1050
+P 1925 1050
+F 0 "#FLG0101" H 1925 1125 50  0001 C CNN
+F 1 "PWR_FLAG" H 1925 1224 50  0000 C CNN
+F 2 "" H 1925 1050 50  0001 C CNN
+F 3 "~" H 1925 1050 50  0001 C CNN
+	1    1925 1050
+	1    0    0    -1
+$EndComp
 $Comp
 L power:PWR_FLAG #FLG0102
@@
 F 2 "Potentiometer_THT:Potentiometer_Piher_T-16H_Single_Horizontal" H 5050 1500 50  0001 C CNN
 F 3 "~" H 5050 1500 50  0001 C CNN
+F 4 "LFO1" H 5050 1500 50  0001 C CNN "Position"
 	1    5050 1500
 	1    0    0    -1
@@
 F 2 "Potentiometer_THT:Potentiometer_Piher_T-16H_Single_Horizontal" H 6200 2025 50  0001 C CNN
 F 3 "~" H 6200 2025 50  0001 C CNN
+F 4 "LFO1" H 6200 2025 50  0001 C CNN "Pos"
 	1    6200 2025
 	1    0    0    -1
@@
 	1150 1375 1150 1650
 Connection ~ 1150 1650
+Text GLabel 1500 1050 1    50   Input ~ 0
+DC-in
+$Comp
+L Sensor_Optical:LDR03 R?
+U 1 1 5C1A1B97
+P 9300 1500
+F 0 "R?" H 9370 1546 50  0000 L CNN
+F 1 "OSC1CV" H 9370 1455 50  0000 L CNN
+F 2 "OptoDevice:R_LDR_10x8.5mm_P7.6mm_Vertical" V 9475 1500 50  0001 C CNN
+F 3 "http://www.elektronica-componenten.nl/WebRoot/StoreNL/Shops/61422969/54F1/BA0C/C664/31B9/2173/C0A8/2AB9/2AEF/LDR03IMP.pdf" H 9300 1450 50  0001 C CNN
+	1    9300 1500
+	1    0    0    -1
+$EndComp
+Wire Wire Line
+	9300 1650 9300 1775
+Connection ~ 9300 1775
+Wire Wire Line
+	9300 1775 8950 1775
+Wire Wire Line
+	9300 1350 9300 1250
+Wire Wire Line
+	9300 1250 9150 1250
+Connection ~ 9150 1250
+$Comp
+L Connector:AudioJack3_Ground J?
+U 1 1 5C1B1418
+P 3050 3600
+F 0 "J?" H 2818 3529 50  0000 R CNN
+F 1 "OSC1CV" H 2818 3620 50  0000 R CNN
+F 2 "Connector_Audio:AudioJack3StereoNarrow-PJ-321" H 3050 3600 50  0001 C CNN
+F 3 "~" H 3050 3600 50  0001 C CNN
+	1    3050 3600
+	-1   0    0    1
+$EndComp
+$Comp
+L Device:R R?
+U 1 1 5C1B1A3B
+P 2675 3400
+F 0 "R?" V 2468 3400 50  0000 C CNN
+F 1 "1k2" V 2559 3400 50  0000 C CNN
+F 2 "Resistor_SMD:R_0805_2012Metric_Pad1.15x1.40mm_HandSolder" V 2605 3400 50  0001 C CNN
+F 3 "~" H 2675 3400 50  0001 C CNN
+	1    2675 3400
+	-1   0    0    1
+$EndComp
+$Comp
+L Device:LED D?
+U 1 1 5C1B1A41
+P 2675 3700
+F 0 "D?" V 2629 3779 50  0000 L CNN
+F 1 "OSC1CV" V 2720 3779 50  0000 L CNN
+F 2 "LED_THT:LED_D3.0mm" H 2675 3700 50  0001 C CNN
+F 3 "~" H 2675 3700 50  0001 C CNN
+	1    2675 3700
+	0    -1   -1   0
+$EndComp
+Wire Wire Line
+	2675 3850 2850 3850
+Wire Wire Line
+	2850 3850 2850 3700
+Wire Wire Line
+	2850 3600 2850 3700
+Connection ~ 2850 3700
+Wire Wire Line
+	2850 3500 2850 3250
+Wire Wire Line
+	2850 3250 2675 3250
+Text GLabel 2850 3250 2    50   Input ~ 0
+OSC1-CV
 $EndSCHEMATC

Commit message: 3D Updated
3D Models
Parts:
- removed J6: AudioJack, Connector_Audio:AudioJack3StereoNarrow-PJ-321, symbol Connector:AudioJack3_Ground
- added TP1: OSC1CV, Connector_Pin:Pin_D1.0mm_L10.0mm_LooseFit, symbol Connector:TestPoint
- gave numbers to parts that had none: 4
Connections:
- net labels added: DC_in, LFO1, LFO2, OSC1, OSC1_CV, OSC2
- net labels removed: DC-in, OSC1-CV
- wire segments 159 -> 156
Changed lines of the file:
@@
 Wire Wire Line
 	2550 2325 2550 2250
-$Comp
-L Connector:AudioJack3_Ground J6
-U 1 1 5C1C640D
-P 1350 2300
-F 0 "J6" H 1118 2229 50  0000 R CNN
-F 1 "AudioJack" H 1118 2320 50  0000 R CNN
-F 2 "Connector_Audio:AudioJack3StereoNarrow-PJ-321" H 1350 2300 50  0001 C CNN
-F 3 "~" H 1350 2300 50  0001 C CNN
-	1    1350 2300
-	1    0    0    1
-$EndComp
-Wire Wire Line
-	1550 2200 1750 2200
 Wire Wire Line
 	2550 2425 1550 2425
-Wire Wire Line
-	1550 2425 1550 2400
 Connection ~ 2550 2425
-Wire Wire Line
-	1550 2400 1550 2300
-Connection ~ 1550 2400
 $Comp
 L Connector:AudioJack3_Ground J8
@@
 Connection ~ 1550 2850
 Connection ~ 1550 2750
-Connection ~ 1550 2425
 $Comp
 L Connector:TestPoint TP5
@@
 	1    0    0    -1
 $EndComp
-Connection ~ 1750 2200
 Wire Wire Line
 	1750 2200 1850 2200
@@
 	1150 1375 1150 1650
 Connection ~ 1150 1650
-Text GLabel 1500 1050 1    50   Input ~ 0
-DC-in
-$Comp
-L Sensor_Optical:LDR03 R?
+$Comp
+L Sensor_Optical:LDR03 R11
 U 1 1 5C1A1B97
 P 9300 1500
-F 0 "R?" H 9370 1546 50  0000 L CNN
+F 0 "R11" H 9370 1546 50  0000 L CNN
 F 1 "OSC1CV" H 9370 1455 50  0000 L CNN
 F 2 "OptoDevice:R_LDR_10x8.5mm_P7.6mm_Vertical" V 9475 1500 50  0001 C CNN
@@
 Connection ~ 9150 1250
 $Comp
-L Connector:AudioJack3_Ground J?
+L Connector:AudioJack3_Ground J4
 U 1 1 5C1B1418
 P 3050 3600
-F 0 "J?" H 2818 3529 50  0000 R CNN
+F 0 "J4" H 2818 3529 50  0000 R CNN
 F 1 "OSC1CV" H 2818 3620 50  0000 R CNN
 F 2 "Connector_Audio:AudioJack3StereoNarrow-PJ-321" H 3050 3600 50  0001 C CNN
@@
 $EndComp
 $Comp
-L Device:R R?
+L Device:R R12
 U 1 1 5C1B1A3B
 P 2675 3400
-F 0 "R?" V 2468 3400 50  0000 C CNN
+F 0 "R12" V 2468 3400 50  0000 C CNN
 F 1 "1k2" V 2559 3400 50  0000 C CNN
 F 2 "Resistor_SMD:R_0805_2012Metric_Pad1.15x1.40mm_HandSolder" V 2605 3400 50  0001 C CNN
@@
 $EndComp
 $Comp
-L Device:LED D?
+L Device:LED D3
 U 1 1 5C1B1A41
 P 2675 3700
-F 0 "D?" V 2629 3779 50  0000 L CNN
+F 0 "D3" V 2629 3779 50  0000 L CNN
 F 1 "OSC1CV" V 2720 3779 50  0000 L CNN
 F 2 "LED_THT:LED_D3.0mm" H 2675 3700 50  0001 C CNN
@@
 Wire Wire Line
 	2850 3250 2675 3250
-Text GLabel 2850 3250 2    50   Input ~ 0
-OSC1-CV
+Text Label 2850 3250 0    50   ~ 0
+OSC1_CV
+Text Label 1175 1050 0    50   ~ 0
+DC_in
+Text Label 5175 1775 0    50   ~ 0
+LFO1
+Text Label 9375 1775 0    50   ~ 0
+OSC1
+Text Label 9125 4025 0    50   ~ 0
+OSC2
+Text Label 5275 4025 0    50   ~ 0
+LFO2
+$Comp
+L Connector:TestPoint TP1
+U 1 1 5C1EB53F
+P 2675 3250
+F 0 "TP1" H 2733 3370 50  0000 L CNN
+F 1 "OSC1CV" H 2733 3279 50  0000 L CNN
+F 2 "Connector_Pin:Pin_D1.0mm_L10.0mm_LooseFit" H 2875 3250 50  0001 C CNN
+F 3 "~" H 2875 3250 50  0001 C CNN
+	1    2675 3250
+	1    0    0    -1
+$EndComp
+Connection ~ 2675 3250
 $EndSCHEMATC
